File: pcb/base_module/rx_mod.brd (EAGLE design)
At the start: 42.5 x 28.8 mm, 29 parts, among them IC1 OPA336N, U1 ATMEGA328

Commit message: pcb oled
Parts:
- added JP5: (no value), SparkFun-Connectors:1X04
Connections:
- net 5V: now also JP5.4
- net GND: now also JP5.3
- net SCL: now also JP5.2
- net SDA: now also JP5.1
Routing:
- net SCL: track 0.00 -> 12.5 mm, vias 0 -> 1
- net SDA: track 0.00 -> 11.5 mm
- net GND: track 170.0 -> 180.8 mm
- net SPI_SEL_B: track 19.0 -> 29.5 mm, vias 3 -> 4
- net CH2: track 33.7 -> 43.1 mm, vias 1 -> 6
- net 5V: track 91.7 -> 100.6 mm, vias 3 -> 4
- net RXVIDOUT2: track 33.7 -> 31.1 mm
- net RESET: track 36.2 -> 38.1 mm, vias 1 -> 3
- net RSSI_B: track 15.3 -> 14.6 mm, vias 1 -> 2
Other:
- board text added: "OLED"
- board text added: "SCL"
- board text added: "SDA"
- board text added: "V4.1"
- board text removed: "V4"
