File: pcb/base_module/rx_mod.brd (EAGLE design)
At the start: 42.5 x 28.8 mm, 29 parts, among them IC1 OPA336N, U1 ATMEGA328

Commit message: new V4.1 base module (I2C OLED pins exposed + some bug fix)
Parts:
- added JP5, JP6: (no value), SparkFun-Connectors:PAD-1.5X4.5
Connections:
- net SCL: now also JP6.P$1
- net SDA: now also JP5.P$1
Routing:
- net GND: track 170.0 -> 186.2 mm, vias 7 -> 10
- net SDA: track 0.00 -> 6.04 mm
- net RESET: track 36.2 -> 40.1 mm
- net SCL: track 0.00 -> 3.64 mm
- net CH2: track 33.7 -> 36.4 mm
Other:
- board text added: "+"
- board text added: "-"
- board text added: "SCL"
- board text added: "SDA"
- board text added: "V4.1"
- board text removed: "V4"
