File: pcb/base_module/rx_mod.sch (EAGLE design)
At the start: 29 parts, among them IC1 OPA336N, U1 ATMEGA328

Commit message: pcb oled
Parts:
- added JP5: (no value), SparkFun-Connectors:M04PTH
Connections:
- net 5V: now also JP5.4
- net GND: now also JP5.3
- net SCL: now also JP5.2
- net SDA: now also JP5.1
Changed lines of the file:
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@@
 <?xml version="1.0" encoding="utf-8"?>
 <!DOCTYPE eagle SYSTEM "eagle.dtd">
-<eagle version="7.5.0">
+<eagle version="7.4.0">
 <drawing>
 <settings>
@@
 <part name="P+5" library="SparkFun" deviceset="3.3V" device="" value="VCC"/>
 <part name="SJ1" library="jumper" deviceset="SJ" device=""/>
+<part name="JP5" library="SparkFun-Connectors" deviceset="M04" device="PTH"/>
+<part name="P+9" library="SparkFun" deviceset="3.3V" device="" value="VCC"/>
+<part name="GND20" library="supply1" deviceset="GND" device=""/>
 </parts>
 <sheets>
@@
 <instance part="P+5" gate="G$1" x="15.24" y="157.48"/>
 <instance part="SJ1" gate="1" x="10.16" y="114.3"/>
+<instance part="JP5" gate="G$1" x="78.74" y="157.48"/>
+<instance part="P+9" gate="G$1" x="93.98" y="165.1"/>
+<instance part="GND20" gate="1" x="93.98" y="154.94"/>
 </instances>
 <busses>
@@
 <pinref part="GND19" gate="1" pin="GND"/>
 </segment>
+<segment>
+<pinref part="JP5" gate="G$1" pin="3"/>
+<pinref part="GND20" gate="1" pin="GND"/>
+<wire x1="83.82" y1="160.02" x2="93.98" y2="160.02" width="0.1524" layer="91"/>
+<wire x1="93.98" y1="160.02" x2="93.98" y2="157.48" width="0.1524" layer="91"/>
+</segment>
 </net>
 <net name="TX" class="0">
@@
 <pinref part="P+5" gate="G$1" pin="3.3V"/>
 </segment>
+<segment>
+<pinref part="JP5" gate="G$1" pin="4"/>
+<pinref part="P+9" gate="G$1" pin="3.3V"/>
+<wire x1="83.82" y1="162.56" x2="93.98" y2="162.56" width="0.1524" layer="91"/>
+<wire x1="93.98" y1="162.56" x2="93.98" y2="165.1" width="0.1524" layer="91"/>
+</segment>
 </net>
 <net name="VIDOUT" class="0">
@@
 <junction x="106.68" y="71.12"/>
 </segment>
+<segment>
+<pinref part="JP5" gate="G$1" pin="2"/>
+<wire x1="83.82" y1="157.48" x2="88.9" y2="157.48" width="0.1524" layer="91"/>
+<label x="83.82" y="157.48" size="1.778" layer="95"/>
+</segment>
 </net>
 <net name="SDA" class="0">
@@
 <junction x="106.68" y="73.66"/>
 </segment>
-</net>
+<segment>
+<pinref part="JP5" gate="G$1" pin="1"/>
+<wire x1="83.82" y1="154.94" x2="88.9" y2="154.94" width="0.1524" layer="91"/>
+<label x="83.82" y="154.94" size="1.778" layer="95"/>
+</segment>
+</net>
