File: pcb/standalone_module/standalone_mod.brd (EAGLE design)
At the start: 31 x 31.2 mm, 11 parts, among them U1 V_REG_317DPACK

Commit message: standalone v2.0
Parts:
- removed R1, R2: (no value), SparkFun-Passives:0805
- removed S1, S2, S3: SWITCH-MOMENTARY-2PTH, SparkFun-Electromechanical:TACTILE-PTH
- removed U1: V_REG_317DPACK, SparkFun-PowerIC:V-REG_DPACK
- added C3: (no value), resistor:E3,5-8
- added D1: (no value), SparkFun-DiscreteSemi:SMA-DIODE
- added JP3: (no value), SparkFun-Connectors:1X03_LONGPADS
- added JP4, JP5: (no value), SparkFun-Connectors:LUXEON-PAD
- added U$1: 7805, #fpv:DDPAK
- added U$2: SKQUCAA010, #fpv:SKQUCAA010
- added U$3: MC001293JACK, #fpv:MC001293
- C1: value (none) -> 0.33uF
- C2: value (none) -> 0.1uF
- moved BATT 28.1 mm to (27.7, 3.39)
- moved JP2 20.4 mm to (39.7, 9.54), turned to 90 degrees
- moved C1 15.6 mm to (12.3, 8.94), turned to 0 degrees
- moved C2 12.2 mm to (11.5, 22.7), turned to 90 degrees
- moved JP1 3.81 mm to (16.4, 18.0)
Connections:
- removed net 3.3V: C2.1, R1.2, U1.4
- removed net N$4: R1.1, R2.2, U1.1
- new net N$2: C3.+, JP1.4
- new net N$3: BATT.2, D1.A, JP3.3
- net 5V: now also C2.1, JP4.P$1, U$1.OUTPUT
- net AUDOUT: now also U$3.3_1, U$3.3_2, U$3.4
- net DOWN: now also U$2.3; no longer S1.1
- net ENTER: now also U$2.6; no longer S2.1
- net GND: now also JP3.1, JP5.P$1, U$1.GND, U$2.4, U$3.1; no longer R2.1, S1.3, S2.3, S3.3
- net N$1: now also D1.C, U$1.INPUT; no longer BATT.2, U1.3
- net UP: now also U$2.1; no longer S3.1
- net VIDOUT: now also C3.-, U$3.2; no longer JP1.4
Routing:
- net AUDOUT: track 14.4 -> 46.0 mm
- net 5V: track 0.00 -> 30.0 mm, vias 0 -> 1
- net N$3: track 0.00 -> 24.7 mm
- net N$2: track 0.00 -> 11.6 mm
- net ENTER: track 12.8 -> 24.4 mm
- net 3.3V: track 11.4 -> 0.00 mm
- net N$4: track 7.38 -> 0.00 mm
- net DOWN: track 24.5 -> 31.4 mm, vias 0 -> 1
- net UP: track 18.3 -> 12.0 mm, vias 1 -> 0
- net VIDOUT: track 18.9 -> 22.1 mm
- net N$1: track 9.30 -> 11.0 mm
Other:
- board size 31 x 31.2 mm -> 46.9 x 31.3 mm
- board text added: "5V"
- board text added: "BATT_2s"
- board text added: "V2.0"
- board text removed: "DOWN"
- board text removed: "ENTER"
- board text removed: "LM317"
- board text removed: "UP"
- board text removed: "V1.0"

Commit message: standalone module v2
Parts:
- added SJ1, SJ2: JUMPER-PAD-2-NC_BY_TRACE, SparkFun-Passives:PAD-JUMPER-2-NC_BY_TRACE_YES_SILK
- JP2: device SparkFun-Connectors:1X03 -> SparkFun-Connectors:1X04
- moved JP2 0.20 mm to (39.8, 9.40)
Connections:
- new net N$4: JP2.4, SJ1.1
- new net N$5: JP2.3, SJ2.1
- net 5V: now also JP2.2
- net AUDOUT: now also SJ2.2; no longer JP2.2
- net VIDOUT: now also SJ1.2; no longer JP2.3
Routing:
- net 5V: track 30.0 -> 56.2 mm
- net AUDOUT: track 46.0 -> 40.8 mm
- net VIDOUT: track 22.1 -> 19.2 mm
- net N$5: track 0.00 -> 2.37 mm
- net N$4: track 0.00 -> 2.30 mm
Other:
- board text removed: "AUDIO"
- board text removed: "VIDEO"
Changed lines of the file:
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@@
 <circle x="3" y="5" radius="3" width="0.4064" layer="42"/>
 <text x="35.75" y="9.04" size="0.8128" layer="25">GND</text>
-<text x="34.74" y="11.73" size="0.8128" layer="25">AUDIO</text>
-<text x="34.88" y="14.12" size="0.8128" layer="25">VIDEO</text>
+<text x="35.96" y="14.77" size="0.8128" layer="25" rot="R180">AUD</text>
+<text x="35.52" y="17.18" size="0.8128" layer="25" rot="R180">VID</text>
 <text x="40.65" y="1.52" size="1.778" layer="25">-</text>
 <text x="32.16" y="1.64" size="1.778" layer="25">+</text>
@@
 <text x="11.15" y="26.56" size="0.8128" layer="25" rot="R180">GND</text>
 <text x="13.65" y="26.66" size="0.8128" layer="25" rot="R180">5V</text>
+<text x="35.85" y="11.64" size="0.8128" layer="25">VCC</text>
 </plain>
 <attributes>
@@
 <attribute name="VALUE" x="12.917" y="21.674" size="0.4064" layer="27" rot="R90"/>
 </element>
-<element name="JP2" library="SparkFun-Connectors" package="1X03" value="" x="39.66" y="9.54" smashed="yes" rot="R90">
-<attribute name="VALUE" x="42.835" y="8.27" size="1.27" layer="27" rot="R90"/>
-</element>
 <element name="U$1" library="#fpv" package="DDPAK" value="7805" x="13.32" y="10.02" smashed="yes" rot="R90"/>
 <element name="U$2" library="#fpv" package="SKQUCAA010" value="SKQUCAA010" x="22.31" y="8.51" smashed="yes"/>
@@
 <attribute name="VALUE" x="13" y="28" size="1.27" layer="27" rot="R90"/>
 </element>
+<element name="JP2" library="SparkFun-Connectors" package="1X04" value="" x="39.8" y="9.4" smashed="yes" rot="R90">
+<attribute name="VALUE" x="42.975" y="8.13" size="1.27" layer="27" rot="R90"/>
+</element>
+<element name="SJ1" library="SparkFun-Passives" package="PAD-JUMPER-2-NC_BY_TRACE_YES_SILK" value="JUMPER-PAD-2-NC_BY_TRACE" x="37" y="17" smashed="yes" rot="R180"/>
+<element name="SJ2" library="SparkFun-Passives" package="PAD-JUMPER-2-NC_BY_TRACE_YES_SILK" value="JUMPER-PAD-2-NC_BY_TRACE" x="37" y="14.4" smashed="yes" rot="R180"/>
 </elements>
 <signals>
@@
 <contactref element="C2" pad="2"/>
 <contactref element="BATT" pad="1"/>
-<contactref element="JP2" pad="1"/>
 <polygon width="0.4064" layer="16" isolate="0.254">
 <vertex x="-5.88" y="1.09"/>
@@
 <via x="5.1" y="13.15" extent="1-16" drill="0.4" shape="square"/>
 <via x="5.1" y="11.15" extent="1-16" drill="0.4" shape="square"/>
-<via x="37.3" y="17.2" extent="1-16" drill="0.4"/>
+<via x="40" y="20.1" extent="1-16" drill="0.4"/>
 <contactref element="U$3" pad="1"/>
 <contactref element="JP5" pad="P$1"/>
+<contactref element="JP2" pad="1"/>
 </signal>
 <signal name="5V">
@@
 <wire x1="13.4" y1="22.5" x2="13.4" y2="28.6" width="0.6096" layer="1"/>
 <wire x1="13.4" y1="28.6" x2="13" y2="29.5" width="0.6096" layer="1"/>
+<contactref element="JP2" pad="2"/>
+<wire x1="33.7" y1="10" x2="27.1" y2="10" width="0.4064" layer="1"/>
+<wire x1="27.1" y1="10" x2="23.7" y2="6.5" width="0.4064" layer="1"/>
+<wire x1="23.7" y1="6.5" x2="17.82" y2="6.5" width="0.4064" layer="1"/>
+<wire x1="17.82" y1="6.5" x2="16.45" y2="7.87" width="0.4064" layer="1"/>
+<wire x1="39.8" y1="11.94" x2="35.64" y2="11.94" width="0.4064" layer="1"/>
+<wire x1="35.64" y1="11.94" x2="33.7" y2="10" width="0.4064" layer="1"/>
 </signal>
 <signal name="VIDOUT">
-<contactref element="JP2" pad="3"/>
 <contactref element="C3" pad="-"/>
 <contactref element="U$3" pad="2"/>
@@
 <wire x1="37.5" y1="24" x2="37.5" y2="20.41" width="0.6096" layer="1"/>
 <wire x1="37.5" y1="20.41" x2="37.49" y2="20.4" width="0.6096" layer="1"/>
-<wire x1="39.66" y1="14.62" x2="39.66" y2="18.23" width="0.6096" layer="1"/>
-<wire x1="39.66" y1="18.23" x2="37.49" y2="20.4" width="0.6096" layer="1"/>
+<contactref element="SJ1" pad="2"/>
+<wire x1="36.492" y1="17" x2="36.492" y2="19.402" width="0.4064" layer="1"/>
+<wire x1="36.492" y1="19.402" x2="37.49" y2="20.4" width="0.4064" layer="1"/>
 </signal>
 <signal name="AUDOUT">
 <contactref element="JP1" pad="5"/>
-<contactref element="JP2" pad="2"/>
 <contactref element="U$3" pad="3_2"/>
 <contactref element="U$3" pad="3_1"/>
@@
 <wire x1="31.79" y1="20.4" x2="31.79" y2="27.95" width="0.6096" layer="16"/>
 <wire x1="31.79" y1="27.95" x2="31.34" y2="28.4" width="0.6096" layer="16"/>
-<wire x1="39.66" y1="12.08" x2="37.32" y2="12.08" width="0.6096" layer="16"/>
-<wire x1="37.32" y1="12.08" x2="36.1" y2="13.3" width="0.6096" layer="16"/>
-<wire x1="36.1" y1="13.3" x2="36.1" y2="15.2" width="0.6096" layer="16"/>
-<wire x1="36.1" y1="15.2" x2="34" y2="17.3" width="0.6096" layer="16"/>
-<wire x1="34" y1="17.3" x2="32.6" y2="17.3" width="0.6096" layer="16"/>
-<wire x1="32.6" y1="17.3" x2="31.8" y2="18.1" width="0.6096" layer="16"/>
-<wire x1="31.8" y1="18.1" x2="31.8" y2="20.39" width="0.6096" layer="16"/>
 <wire x1="31.8" y1="20.39" x2="31.79" y2="20.4" width="0.6096" layer="16"/>
+<contactref element="SJ2" pad="2"/>
+<wire x1="36.492" y1="14.4" x2="35.5" y2="14.4" width="0.4064" layer="1"/>
+<wire x1="31.9" y1="18" x2="31.9" y2="20.29" width="0.4064" layer="1"/>
+<wire x1="31.9" y1="20.29" x2="31.79" y2="20.4" width="0.4064" layer="1"/>
+<wire x1="31.9" y1="18" x2="35.5" y2="14.4" width="0.4064" layer="1"/>
 </signal>
 <signal name="N$1">
@@
 <wire x1="33.87" y1="4.18" x2="34.62" y2="3.13" width="0.6096" layer="1"/>
 </signal>
+<signal name="N$4">
+<contactref element="SJ1" pad="1"/>
+<contactref element="JP2" pad="4"/>
+<wire x1="39.8" y1="17.02" x2="37.528" y2="17.02" width="0.4064" layer="1"/>
+<wire x1="37.528" y1="17.02" x2="37.508" y2="17" width="0.4064" layer="1"/>
+</signal>
+<signal name="N$5">
+<contactref element="SJ2" pad="1"/>
+<contactref element="JP2" pad="3"/>
+<wire x1="39.8" y1="14.48" x2="37.508" y2="14.48" width="0.4064" layer="1"/>
+<wire x1="37.508" y1="14.48" x2="37.508" y2="14.4" width="0.4064" layer="1"/>
+</signal>
 </signals>
