File: pcb/diversity_module/div_mod.brd (EAGLE design)
At the start: 40 x 29 mm, 17 parts, among them IC3 OPA336N

Commit message: diversity module v2.2 - better traces and big holes for battery
Parts:
- removed SJ1: (no value), jumper:SJ
- JP2: device SparkFun-Connectors:1X02_LOCK -> SparkFun-Connectors:1X02
- moved R1 19.2 mm to (35.5, 7.13)
- moved JP2 0.48 mm to (38.8, 26.3)
Connections:
- net 5V: no longer SJ1.2
- net ENABLE_P: no longer SJ1.1
Routing:
- net GND: track 135.8 -> 96.7 mm, vias 8 -> 7
- net N$1: track 24.9 -> 5.85 mm
- net SPI_SEL_B: track 49.5 -> 41.5 mm, vias 4 -> 1
- net 5V: track 65.4 -> 62.1 mm
- net ENABLE_P: track 64.6 -> 62.7 mm
- net RXVIDOUT2: track 46.9 -> 45.3 mm, vias 3 -> 2
- net SPI_DATA: track 48.8 -> 47.9 mm
- net RSSI_MOD: track 28.0 -> 27.3 mm
Other:
- board text added: "mikym0use diversity module v2.2 part of JAFar project"
- board text removed: "mikym0use diversity module v2.1 part of JAFar project"
- board text removed: "power"

Commit message: div mod updates
Parts:
- R3: value 10k -> 100k
- R4: value 100k -> 10k
Changed lines of the file:
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@@
 <attribute name="VALUE" x="30.92" y="22.91" size="1.27" layer="27"/>
 </element>
-<element name="R3" library="SparkFun-Passives" package="0805" value="10k" x="13.28" y="19.13" smashed="yes" rot="MR90">
+<element name="R3" library="SparkFun-Passives" package="0805" value="100k" x="13.28" y="19.13" smashed="yes" rot="MR90">
 <attribute name="NAME" x="12.8755" y="16.248" size="0.8128" layer="26" font="vector" rot="MR90"/>
 <attribute name="VALUE" x="11.713" y="18.304" size="0.8128" layer="28" font="vector" rot="MR90"/>
@@
 <attribute name="VALUE" x="40.02" y="29.515" size="1.27" layer="27" rot="R180"/>
 </element>
-<element name="R4" library="SparkFun-Passives" package="0805" value="100k" x="13.29" y="22.78" smashed="yes" rot="MR90">
+<element name="R4" library="SparkFun-Passives" package="0805" value="10k" x="13.29" y="22.78" smashed="yes" rot="MR90">
 <attribute name="NAME" x="14.1155" y="22.018" size="0.8128" layer="26" font="vector" rot="MR90"/>
 <attribute name="VALUE" x="11.513" y="21.534" size="0.8128" layer="28" font="vector" rot="MR90"/>
@@
 </polygon>
 <polygon width="0.254" layer="16" isolate="0.254">
-<vertex x="0" y="0"/>
+<vertex x="2" y="-0.08"/>
 <vertex x="42" y="0"/>
 <vertex x="42" y="28"/>
-<vertex x="0" y="28"/>
+<vertex x="10.63" y="28.44"/>
+<vertex x="10.45" y="27.91"/>
+<vertex x="10.53" y="8.9"/>
+<vertex x="2" y="8.98"/>
+<vertex x="1.91" y="8.3"/>
 </polygon>
 <polygon width="0.4064" layer="1" isolate="0.4064">
