File: pcb/diversity_module/div_mod.sch (EAGLE design)
At the start: 17 parts, among them IC3 OPA336N

Commit message: diversity module v2.2 - better traces and big holes for battery
Parts:
- removed SJ1: (no value), jumper:SJ
- JP2: device SparkFun-Connectors:M02LOCK -> SparkFun-Connectors:M02PTH
Connections:
- net 5V: no longer SJ1.2
- net ENABLE_P: no longer SJ1.1
Other:
- note removed: "power"
Changed lines of the file:
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@@
 <?xml version="1.0" encoding="utf-8"?>
 <!DOCTYPE eagle SYSTEM "eagle.dtd">
-<eagle version="7.5.0">
+<eagle version="7.7.0">
 <drawing>
 <settings>
@@
 <part name="C2" library="SparkFun-Capacitors" deviceset="CAP" device="0805" value="1uf"/>
 <part name="GND2" library="supply1" deviceset="GND" device=""/>
-<part name="JP2" library="SparkFun-Connectors" deviceset="M02" device="LOCK"/>
+<part name="JP2" library="SparkFun-Connectors" deviceset="M02" device="PTH"/>
 <part name="GND12" library="supply1" deviceset="GND" device=""/>
-<part name="SJ1" library="jumper" deviceset="SJ" device=""/>
-<part name="P+1" library="SparkFun" deviceset="3.3V" device="" value="VCC"/>
 <part name="R4" library="SparkFun-Passives" deviceset="RESISTOR" device="0805-RES" value="100k"/>
 </parts>
@@
 <text x="111.76" y="111.76" size="1.778" layer="97">buffer bypass</text>
 <text x="119.38" y="78.74" size="1.778" layer="95">OPA337</text>
-<text x="106.68" y="38.1" size="1.778" layer="97">power</text>
 </plain>
 <instances>
@@
 <instance part="JP2" gate="G$1" x="162.56" y="91.44"/>
 <instance part="GND12" gate="1" x="182.88" y="86.36"/>
-<instance part="SJ1" gate="1" x="114.3" y="43.18"/>
-<instance part="P+1" gate="G$1" x="134.62" y="48.26"/>
 <instance part="R4" gate="G$1" x="213.36" y="147.32" rot="R180"/>
 </instances>
@@
 <pinref part="P+5" gate="G$1" pin="3.3V"/>
 </segment>
-<segment>
-<pinref part="SJ1" gate="1" pin="2"/>
-<wire x1="119.38" y1="43.18" x2="134.62" y2="43.18" width="0.1524" layer="91"/>
-<pinref part="P+1" gate="G$1" pin="3.3V"/>
-<wire x1="134.62" y1="43.18" x2="134.62" y2="48.26" width="0.1524" layer="91"/>
-</segment>
 </net>
 <net name="AUDOUT" class="0">
@@
 <label x="195.58" y="147.32" size="1.778" layer="95"/>
 </segment>
-<segment>
-<pinref part="SJ1" gate="1" pin="1"/>
-<wire x1="109.22" y1="43.18" x2="88.9" y2="43.18" width="0.1524" layer="91"/>
-<label x="93.98" y="43.18" size="1.778" layer="95"/>
-</segment>
-</net>
+</net>

Commit message: div mod updates
Parts:
- R3: value 10k -> 100k
- R4: value 100k -> 10k
Changed lines of the file:
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@@
 <part name="P+3" library="SparkFun" deviceset="3.3V" device="" value="VCC"/>
 <part name="GND6" library="supply1" deviceset="GND" device=""/>
-<part name="R3" library="SparkFun-Passives" deviceset="RESISTOR" device="0805-RES" value="10k"/>
+<part name="R3" library="SparkFun-Passives" deviceset="RESISTOR" device="0805-RES" value="100k"/>
 <part name="GND7" library="supply1" deviceset="GND" device=""/>
 <part name="IC3" library="burr-brown" deviceset="OPA336" device="N"/>
@@
 <part name="JP2" library="SparkFun-Connectors" deviceset="M02" device="PTH"/>
 <part name="GND12" library="supply1" deviceset="GND" device=""/>
-<part name="R4" library="SparkFun-Passives" deviceset="RESISTOR" device="0805-RES" value="100k"/>
+<part name="R4" library="SparkFun-Passives" deviceset="RESISTOR" device="0805-RES" value="10k"/>
 </parts>
 <sheets>
